File: circuit/light-panel/light-panel.kicad_pcb (KiCad board)
At the start: 2 copper layers, 12 parts, among them J1 Screw_Terminal_01x02

Commit message: start layout
Parts:
- added D10: KT-0603R, LED_SMD:LED_0603_1608Metric, F.Cu at (143.6, 101.1)
- added D11: KT-0603R, LED_SMD:LED_0603_1608Metric, F.Cu at (147.6, 93.3)
- added D12: KT-0603R, LED_SMD:LED_0603_1608Metric, F.Cu at (147.6, 95.9)
- added D13: KT-0603R, LED_SMD:LED_0603_1608Metric, F.Cu at (147.6, 98.5)
- added D14: KT-0603R, LED_SMD:LED_0603_1608Metric, F.Cu at (147.6, 101.1)
- added D15: KT-0603R, LED_SMD:LED_0603_1608Metric, F.Cu at (151.7, 93.3)
- added D16: KT-0603R, LED_SMD:LED_0603_1608Metric, F.Cu at (151.7, 95.9)
- added D17: KT-0603R, LED_SMD:LED_0603_1608Metric, F.Cu at (151.7, 98.5)
- added D18: KT-0603R, LED_SMD:LED_0603_1608Metric, F.Cu at (151.7, 101.1)
- added D7: KT-0603R, LED_SMD:LED_0603_1608Metric, F.Cu at (143.6, 93.3)
- added D8: KT-0603R, LED_SMD:LED_0603_1608Metric, F.Cu at (143.6, 95.9)
- added D9: KT-0603R, LED_SMD:LED_0603_1608Metric, F.Cu at (143.6, 98.5)
- added R2: 330Ω, Resistor_SMD:R_0603_1608Metric, F.Cu at (139.5, 93.3)
- added R3: 330Ω, Resistor_SMD:R_0603_1608Metric, F.Cu at (139.5, 95.8)
- added R4: 330Ω, Resistor_SMD:R_0603_1608Metric, F.Cu at (139.5, 98.3)
- added R5: 330Ω, Resistor_SMD:R_0603_1608Metric, F.Cu at (139.5, 100.8)
- added R6: 330Ω, Resistor_SMD:R_0603_1608Metric, F.Cu at (139.5, 103.3)
- added R7: 330Ω, Resistor_SMD:R_0603_1608Metric, F.Cu at (139.5, 105.8)
- added R8: 330Ω, Resistor_SMD:R_0603_1608Metric, F.Cu at (139.5, 108.3)
- added R9: 330Ω, Resistor_SMD:R_0603_1608Metric, F.Cu at (139.5, 110.8)
- R1: value 220Ω -> 330Ω
- moved D1 40.5 mm to (97.7, 108.0)
- moved D2 27.9 mm to (104.0, 99.5)
- moved D4 26.7 mm to (104.2, 103.5)
- moved D6 25.6 mm to (104.2, 107.5)
- moved D3 24.1 mm to (108.5, 99.5)
- moved D5 23.0 mm to (108.3, 103.5)
