File: circuit/light-panel/light-panel.kicad_sch (KiCad schematic)
At the start: 35 parts, among them J1 Screw_Terminal_01x02

Commit message: rearrange leds
Parts:
- added TP1, TP2, TP3: TestPoint_Probe, TestPoint:TestPoint_THTPad_1.0x1.0mm_Drill0.5mm, symbol Connector:TestPoint_Probe
Connections:
- net +5V: now also TP2.1
- net GND: now also TP3.1
- net at D3.1 (K), D4.2 (A): now also TP1.1
